File: pcb/rcl_mini.brd (EAGLE design)
At the start: 160 x 100 mm, 59 parts, among them CN1 USB mini B, Q1 8MHz, Q2 IRLML5203, U1 MCP6002T-I/SN, U2 MCP6002T-I/SN, U3 MCP6002T-I/SN, U4 STM32F100CBT6, U5 MCP73831/OT, U6 MCP1703CB, X1 BAT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

Commit message: pcb v1.0
Parts:
- moved C4 11.4 mm to (15.2, 76.2), turned to 0 degrees
- moved R4 10.2 mm to (14.0, 72.4), turned to 90 degrees
- moved C6 9.14 mm to (17.7, 65.0), turned to 180 degrees
- moved C7 8.82 mm to (16.6, 55.9), turned to 270 degrees
- moved C18 5.97 mm to (18.2, 73.7), turned to 180 degrees
- moved U1 5.24 mm to (17.8, 68.6), turned to 0 degrees
- moved C5 4.58 mm to (22.9, 73.7)
- moved C19 4.27 mm to (18.2, 71.1), turned to 180 degrees
- moved R9 2.81 mm to (18.9, 55.9)
- moved R8 1.44 mm to (21.8, 65.0), turned to 0 degrees
Routing:
- net GND: track 0.00 -> 27.5 mm
- net VCC_OPAMP: track 0.00 -> 8.89 mm
- net LPOT: track 0.00 -> 7.77 mm
- net LCUR2: track 0.00 -> 6.21 mm
- net N$10: track 0.00 -> 5.80 mm
- net N$6: track 0.00 -> 5.66 mm
- net HCUR2: track 0.00 -> 5.54 mm
- net LCUR: track 0.00 -> 5.40 mm
- net N$16: track 0.00 -> 4.51 mm
- net N$11: track 0.00 -> 4.37 mm
- net HCUR: track 0.00 -> 4.13 mm
- net PA2: track 0.00 -> 3.25 mm
- net PA1: track 0.00 -> 2.99 mm

Commit message: pcb v1.0
Parts:
- added R18, R19: 4.7k, rcl:M0805
- moved CN1 134.2 mm to (66.0, 95.2), turned to 90 degrees
- moved S3 128.2 mm to (53.3, 41.9)
- moved Q1 126.9 mm to (52.1, 74.9), turned to 90 degrees
- moved R1 123.7 mm to (58.4, 96.5), turned to 90 degrees
- moved C1 121.3 mm to (45.5, 95.6), turned to 90 degrees
- moved R2 121.0 mm to (49.5, 99.1)
- moved U5 110.3 mm to (49.5, 96.5), turned to 270 degrees
- moved L1 106.5 mm to (38.5, 75.3), turned to 180 degrees
- moved S2 106.4 mm to (41.9, 41.9)
- moved U6 103.0 mm to (35.6, 92.7)
- moved X1 101.6 mm to (40.6, 96.5)
- moved X3 100.4 mm to (39.4, 83.8)
- moved R13 99.5 mm to (30.4, 66.7), turned to 180 degrees
- moved LED1 93.8 mm to (55.9, 99.1), turned to 90 degrees
- moved C17 93.1 mm to (41.8, 52.7), turned to 180 degrees
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Connections:
- net OLED_I2C_SCK: now also R19.2
- net OLED_I2C_SDA: now also R18.2
- net VDD: now also R18.1, R19.1
Routing:
- net GND: track 27.5 -> 366.8 mm, vias 0 -> 10
- net VDD: track 0.00 -> 105.7 mm, vias 0 -> 1
- net VCC_OPAMP: track 8.89 -> 62.0 mm, vias 0 -> 4
- net N$20: track 0.00 -> 52.6 mm, vias 0 -> 4
- net SWCLK: track 0.00 -> 44.7 mm
- net OLED_I2C_SCK: track 0.00 -> 39.9 mm, vias 0 -> 2
- net SW1: track 0.00 -> 39.7 mm, vias 0 -> 1
- net SWDIO: track 0.00 -> 34.2 mm
- net PA1: track 2.99 -> 37.0 mm
- net OLED_I2C_SDA: track 0.00 -> 31.4 mm, vias 0 -> 1
- net SW3: track 0.00 -> 29.4 mm
- net UART_RX: track 0.00 -> 29.4 mm
- net SW2: track 0.00 -> 27.8 mm
- net UART_TX: track 0.00 -> 27.6 mm
- net N$24: track 0.00 -> 26.5 mm
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Other:
- board size 160 x 100 mm -> 66 x 68.2 mm
