File: pcb/rcl_mini.brd (EAGLE design)
At the start: 77.5 x 64.4 mm, 60 parts, among them CN1 USB mini B, Q1 8MHz, Q2 IRLML5203, U1 MCP6002T-I/SN, U2 MCP6002T-I/SN, U3 MCP6002T-I/SN, U4 STM32F100CBT6, U5 MCP73831/OT, U6 MCP1703CB, X1 BAT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

Commit message: pcb design improvements
Routing:
- net N$7: track 16.9 -> 18.5 mm
Changed lines of the file:
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@@
 <contactref element="X2" pad="1"/>
 <wire x1="24.2078" y1="58.585" x2="23.025" y2="58.585" width="0.4064" layer="1"/>
-<wire x1="23.025" y1="58.585" x2="19.05" y2="54.61" width="0.4064" layer="1"/>
-<wire x1="19.05" y1="54.61" x2="15.367" y2="54.61" width="1.27" layer="1"/>
-<wire x1="15.367" y1="54.61" x2="14.605" y2="53.848" width="0.4064" layer="1"/>
+<wire x1="23.025" y1="58.585" x2="17.35" y2="53.91" width="0.4064" layer="1"/>
+<wire x1="17.35" y1="53.91" x2="13.667" y2="53.91" width="1.27" layer="1"/>
+<wire x1="13.667" y1="53.91" x2="14.605" y2="53.848" width="0.4064" layer="1"/>
 <wire x1="14.605" y1="53.848" x2="12.748" y2="53.848" width="1.778" layer="1"/>
 <wire x1="12.748" y1="53.848" x2="12.7" y2="53.8" width="1.778" layer="1"/>
