File: pcb/rcl_mini.sch (EAGLE design)
At the start: 58 parts, among them CN1 USB mini B, Q1 8MHz, Q2 IRLML5203, U1 MCP6002T-I/SN, U2 MCP6002T-I/SN, U3 MCP6002T-I/SN, U4 STM32F100CBT6, U5 MCP73831/OT, U6 MCP1703CB, X1 BAT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

Commit message: pcb v1.0
Parts:
- added R17: 10k, rcl:R-EU_M0805
Connections:
- new net N$1: R17.1, U4.PB2
- net GND: now also R17.2
Changed lines of the file:
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@@
 <part name="SUPPLY1" library="supply2" deviceset="+4.1V" device=""/>
 <part name="SUPPLY2" library="supply2" deviceset="+4.1V" device=""/>
+<part name="R17" library="rcl" deviceset="R-EU_" device="M0805" value="10k"/>
+<part name="GND20" library="supply1" deviceset="GND" device=""/>
 </parts>
 <sheets>
@@
 <instance part="SUPPLY1" gate="P" x="50.8" y="262.89"/>
 <instance part="SUPPLY2" gate="P" x="201.93" y="190.5"/>
+<instance part="R17" gate="G$1" x="129.54" y="165.1"/>
+<instance part="GND20" gate="1" x="138.43" y="160.02"/>
 </instances>
 <busses>
@@
 <wire x1="-38.1" y1="204.47" x2="-44.45" y2="204.47" width="0.1524" layer="91"/>
 <junction x="-44.45" y="204.47"/>
+</segment>
+<segment>
+<pinref part="R17" gate="G$1" pin="2"/>
+<pinref part="GND20" gate="1" pin="GND"/>
+<wire x1="134.62" y1="165.1" x2="138.43" y2="165.1" width="0.1524" layer="91"/>
+<wire x1="138.43" y1="165.1" x2="138.43" y2="162.56" width="0.1524" layer="91"/>
 </segment>
 </net>
@@
 </segment>
 </net>
+<net name="N$1" class="0">
+<segment>
+<pinref part="U4" gate="G$1" pin="PB2"/>
+<pinref part="R17" gate="G$1" pin="1"/>
+<wire x1="120.65" y1="165.1" x2="124.46" y2="165.1" width="0.1524" layer="91"/>
+</segment>
+</net>

Commit message: pcb v1.0
Parts:
- R6, R7: value 100 -> 150
Connections:
- net N$13 renamed NRST
- net N$14 renamed PA3
- net N$18 renamed PA5
- net N$22 renamed PA7
- net N$7 renamed PA4
- net N$8 renamed PA2
- net N$9 renamed PA1
Changed lines of the file:
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@@
 <part name="GND6" library="supply1" deviceset="GND" device=""/>
 <part name="GND7" library="supply1" deviceset="GND" device=""/>
-<part name="R6" library="rcl" deviceset="R-EU_" device="M0805" value="100"/>
-<part name="R7" library="rcl" deviceset="R-EU_" device="M0805" value="100"/>
+<part name="R6" library="rcl" deviceset="R-EU_" device="M0805" value="150"/>
+<part name="R7" library="rcl" deviceset="R-EU_" device="M0805" value="150"/>
 <part name="GND8" library="supply1" deviceset="GND" device=""/>
 <part name="C6" library="rcl" deviceset="C-EU" device="C0805" value="470p"/>
@@
 </segment>
 </net>
-<net name="N$9" class="0">
+<net name="PA1" class="0">
 <segment>
 <pinref part="U4" gate="G$1" pin="PA1"/>
@@
 </segment>
 </net>
-<net name="N$8" class="0">
+<net name="PA2" class="0">
 <segment>
 <pinref part="R5" gate="G$1" pin="2"/>
@@
 </segment>
 </net>
-<net name="N$7" class="0">
+<net name="PA4" class="0">
 <segment>
 <pinref part="U4" gate="G$1" pin="PA4"/>
@@
 </segment>
 </net>
-<net name="N$18" class="0">
+<net name="PA5" class="0">
 <segment>
 <pinref part="U4" gate="G$1" pin="PA5"/>
@@
 </segment>
 </net>
-<net name="N$22" class="0">
+<net name="PA7" class="0">
 <segment>
 <pinref part="U4" gate="G$1" pin="PA7"/>
@@
 </segment>
 </net>
-<net name="N$13" class="0">
+<net name="NRST" class="0">
 <segment>
 <pinref part="U4" gate="G$1" pin="NRST"/>
@@
 </segment>
 </net>
-<net name="N$14" class="0">
+<net name="PA3" class="0">
 <segment>
 <pinref part="U4" gate="G$1" pin="PA3"/>

Commit message: pcb v1.0
Parts:
- added R18, R19: 4.7k, rcl:R-EU_M0805
Connections:
- net OLED_I2C_SCK: now also R19.2
- net OLED_I2C_SDA: now also R18.2
- net VDD: now also R18.1, R19.1
